Commit message: Use MuJoCo simulation and add Rerun inspection

File: examples/adapters/planar.urdf (robot description, URDF)
Before this commit: robot planar-example, 4 links, 3 joints
Links:
- link forearm: mass None -> 0.1; geometry collision box size=0.15 0.02 0.02; visual box size=0.15 0.02 0.02
- link upper: mass None -> 0.15; geometry collision box size=0.2 0.02 0.02; visual box size=0.2 0.02 0.02
